File: SimpleF303.sch (KiCad schematic (older format))
At the start: 28 parts, among them J1 47346-0001, J2 Conn_01x20_Male, J3 Conn_01x20_Male, SW1 B3U-1000P, U1 AZ1117CH-3.3TRG1, U2 STM32F303CCT6, Y1 8Mhz 20pf

Commit message: clearly I can't get some parts so I change selection
Parts:
- C1, C5, C6, C7, C9: LCSC C24452 -> C307348; Part Number CL10B104JB8NNNC -> CL10B104KB8WPNC
- SW1: value B3U-1000P -> K2-1187SQ-A4SW-06; footprint Button_Switch_SMD:SW_SPST_B3U-1000P -> KiCad:K2-1187SQ-A4SW-06; LCSC C231329 -> C92584; Part Number B3U-1000P -> K2-1187SQ-A4SW-06
Changed lines of the file:
@@
 F 2 "Capacitor_SMD:C_0603_1608Metric" H 2188 6850 50  0001 C CNN
 F 3 "~" H 2150 7000 50  0001 C CNN
-F 4 "C24452" H 2150 7000 50  0001 C CNN "LCSC"
-F 5 "CL10B104JB8NNNC" H 2150 7000 50  0001 C CNN "Part Number"
+F 4 "C307348" H 2150 7000 50  0001 C CNN "LCSC"
+F 5 "CL10B104KB8WPNC" H 2150 7000 50  0001 C CNN "Part Number"
 	1    2150 7000
 	1    0    0    -1
@@
 F 2 "Capacitor_SMD:C_0603_1608Metric" H 1738 6850 50  0001 C CNN
 F 3 "~" H 1700 7000 50  0001 C CNN
-F 4 "C24452" H 1700 7000 50  0001 C CNN "LCSC"
-F 5 "CL10B104JB8NNNC" H 1700 7000 50  0001 C CNN "Part Number"
+F 4 "C307348" H 1700 7000 50  0001 C CNN "LCSC"
+F 5 "CL10B104KB8WPNC" H 1700 7000 50  0001 C CNN "Part Number"
 	1    1700 7000
 	1    0    0    -1
@@
 F 2 "Capacitor_SMD:C_0603_1608Metric" H 1288 6850 50  0001 C CNN
 F 3 "~" H 1250 7000 50  0001 C CNN
-F 4 "C24452" H 1250 7000 50  0001 C CNN "LCSC"
-F 5 "CL10B104JB8NNNC" H 1250 7000 50  0001 C CNN "Part Number"
+F 4 "C307348" H 1250 7000 50  0001 C CNN "LCSC"
+F 5 "CL10B104KB8WPNC" H 1250 7000 50  0001 C CNN "Part Number"
 	1    1250 7000
 	1    0    0    -1
@@
 F 2 "Capacitor_SMD:C_0603_1608Metric" H 838 6850 50  0001 C CNN
 F 3 "~" H 800 7000 50  0001 C CNN
-F 4 "C24452" H 800 7000 50  0001 C CNN "LCSC"
-F 5 "CL10B104JB8NNNC" H 800 7000 50  0001 C CNN "Part Number"
+F 4 "C307348" H 800 7000 50  0001 C CNN "LCSC"
+F 5 "CL10B104KB8WPNC" H 800 7000 50  0001 C CNN "Part Number"
 	1    800  7000
 	1    0    0    -1
@@
 F 2 "Capacitor_SMD:C_0603_1608Metric" H 1238 1100 50  0001 C CNN
 F 3 "~" H 1200 1250 50  0001 C CNN
-F 4 "C24452" H 1200 1250 50  0001 C CNN "LCSC"
-F 5 "CL10B104JB8NNNC" H 1200 1250 50  0001 C CNN "Part Number"
+F 4 "C307348" H 1200 1250 50  0001 C CNN "LCSC"
+F 5 "CL10B104KB8WPNC" H 1200 1250 50  0001 C CNN "Part Number"
 	1    1200 1250
 	1    0    0    -1
@@
 P 1500 1500
 F 0 "SW1" V 1454 1630 50  0000 L CNN
-F 1 "B3U-1000P" V 1545 1630 50  0000 L CNN
-F 2 "Button_Switch_SMD:SW_SPST_B3U-1000P" H 1500 1500 50  0001 C CNN
+F 1 "K2-1187SQ-A4SW-06" V 1545 1630 50  0000 L CNN
+F 2 "KiCad:K2-1187SQ-A4SW-06" H 1500 1500 50  0001 C CNN
 F 3 "https://omronfs.omron.com/en_US/ecb/products/pdf/en-b3u.pdf" H 1500 1500 50  0001 C CNN
-F 4 "B3U-1000P" H 1500 1500 50  0001 C CNN "Part Number"
-F 5 "C231329" H 1500 1500 50  0001 C CNN "LCSC"
+F 4 "K2-1187SQ-A4SW-06" H 1500 1500 50  0001 C CNN "Part Number"
+F 5 "C92584" H 1500 1500 50  0001 C CNN "LCSC"
 	1    1500 1500
 	-1   0    0    1

Commit message: small changes
Parts:
- added U?: STM32F103C8Tx, Package_QFP:LQFP-48_7x7mm_P0.5mm, symbol MCU_ST_STM32F1:STM32F103C8Tx
- C2: LCSC C77040 -> C38898; Part Number GRM188R60J106KE47D -> 0603X106K100NT
Connections:
- net BOOT0: now also J2.3 (Pin_3); no longer J2.4 (Pin_4)
- net NRST: now also J3.2 (Pin_2); no longer J2.3 (Pin_3)
- net PA0: now also J2.17 (Pin_17); no longer J2.18 (Pin_18)
- net PA1: now also J2.18 (Pin_18); no longer J2.19 (Pin_19)
- net PA10: now also J3.3 (Pin_3); no longer J3.2 (Pin_2)
- net PA13: now also J2.4 (Pin_4); no longer J2.5 (Pin_5)
- net PA14: now also J2.5 (Pin_5); no longer J2.6 (Pin_6)
- net PA15: now also J2.6 (Pin_6); no longer J2.7 (Pin_7)
- net PA2: now also J2.19 (Pin_19); no longer J3.19 (Pin_19)
- net PA3: now also J3.19 (Pin_19); no longer J3.18 (Pin_18)
- net PA4: now also J3.18 (Pin_18); no longer J3.17 (Pin_17)
- net PA5: now also J3.17 (Pin_17); no longer J3.16 (Pin_16)
- net PA6: now also J3.16 (Pin_16); no longer J3.15 (Pin_15)
- net PA7: now also J3.15 (Pin_15); no longer J3.14 (Pin_14)
- net PA8: now also J3.5 (Pin_5); no longer J3.4 (Pin_4)
- net PA9: now also J3.4 (Pin_4); no longer J3.3 (Pin_3)
- net PB0: now also J3.14 (Pin_14); no longer J3.13 (Pin_13)
- net PB1: now also J3.13 (Pin_13); no longer J3.12 (Pin_12)
- net PB10: now also J3.11 (Pin_11); no longer J3.10 (Pin_10)
- net PB11: now also J3.10 (Pin_10); no longer J3.9 (Pin_9)
- net PB12: now also J3.9 (Pin_9); no longer J3.8 (Pin_8)
- net PB13: now also J3.8 (Pin_8); no longer J3.7 (Pin_7)
- net PB14: now also J3.7 (Pin_7); no longer J3.6 (Pin_6)
- net PB15: now also J3.6 (Pin_6); no longer J3.5 (Pin_5)
- net PB2: now also J3.12 (Pin_12); no longer J3.11 (Pin_11)
- net PB3: now also J2.7 (Pin_7); no longer J2.8 (Pin_8)
- net PB4: now also J2.8 (Pin_8); no longer J2.9 (Pin_9)
- net PB5: now also J2.9 (Pin_9); no longer J2.10 (Pin_10)
- net PB6: now also J2.10 (Pin_10); no longer J2.11 (Pin_11)
- net PB7: now also J2.11 (Pin_11); no longer J2.12 (Pin_12)
- net PB8: now also J2.12 (Pin_12); no longer J2.13 (Pin_13)
- net PB9: now also J2.13 (Pin_13); no longer J2.14 (Pin_14)
- net PC13: now also J2.14 (Pin_14); no longer J2.15 (Pin_15)
- net PC14: now also J2.15 (Pin_15); no longer J2.16 (Pin_16)
- net PC15: now also J2.16 (Pin_16); no longer J2.17 (Pin_17)
Other:
- note added: "U don't need most of them if u use F103\n"
- moved on the sheet: SW1
Changed lines of the file:
@@
 	1    0    0    -1
 $EndComp
-Wire Notes Line
-	3900 6400 3900 7650
-Wire Notes Line
-	600  6400 3900 6400
-Wire Notes Line
-	600  7650 3900 7650
 Wire Wire Line
 	3500 6650 3500 6850
@@
 Connection ~ 1000 5650
 Wire Wire Line
-	1200 1400 1200 1500
-Connection ~ 1200 1500
-Wire Wire Line
-	1200 1500 1200 1750
-Wire Wire Line
 	1200 1100 800  1100
 Wire Wire Line
@@
 L power:GND #PWR010
 U 1 1 5E235A77
-P 1800 1500
-F 0 "#PWR010" H 1800 1250 50  0001 C CNN
-F 1 "GND" V 1805 1372 50  0000 R CNN
-F 2 "" H 1800 1500 50  0001 C CNN
-F 3 "" H 1800 1500 50  0001 C CNN
-	1    1800 1500
+P 1800 1400
+F 0 "#PWR010" H 1800 1150 50  0001 C CNN
+F 1 "GND" V 1805 1272 50  0000 R CNN
+F 2 "" H 1800 1400 50  0001 C CNN
+F 3 "" H 1800 1400 50  0001 C CNN
+	1    1800 1400
 	0    -1   -1   0
 $EndComp
@@
 L Switch:SW_DIP_x01 SW1
 U 1 1 5E234436
-P 1500 1500
-F 0 "SW1" V 1454 1630 50  0000 L CNN
-F 1 "K2-1187SQ-A4SW-06" V 1545 1630 50  0000 L CNN
-F 2 "KiCad:K2-1187SQ-A4SW-06" H 1500 1500 50  0001 C CNN
-F 3 "https://omronfs.omron.com/en_US/ecb/products/pdf/en-b3u.pdf" H 1500 1500 50  0001 C CNN
-F 4 "K2-1187SQ-A4SW-06" H 1500 1500 50  0001 C CNN "Part Number"
-F 5 "C92584" H 1500 1500 50  0001 C CNN "LCSC"
-	1    1500 1500
+P 1500 1400
+F 0 "SW1" V 1454 1530 50  0000 L CNN
+F 1 "K2-1187SQ-A4SW-06" V 1545 1530 50  0000 L CNN
+F 2 "KiCad:K2-1187SQ-A4SW-06" H 1500 1400 50  0001 C CNN
+F 3 "https://omronfs.omron.com/en_US/ecb/products/pdf/en-b3u.pdf" H 1500 1400 50  0001 C CNN
+F 4 "K2-1187SQ-A4SW-06" H 1500 1400 50  0001 C CNN "Part Number"
+F 5 "C92584" H 1500 1400 50  0001 C CNN "LCSC"
+	1    1500 1400
 	-1   0    0    1
 $EndComp
@@
 Wire Wire Line
 	5700 4400 5300 4400
+Text Label 5700 2600 2    50   ~ 0
+NRST
 Text Label 4350 2700 0    50   ~ 0
-NRST
-Text Label 4350 2800 0    50   ~ 0
 BOOT0
 $Comp
@@
 F 2 "Capacitor_SMD:C_0603_1608Metric" H 988 4350 50  0001 C CNN
 F 3 "~" H 950 4500 50  0001 C CNN
-F 4 "C77040" H 950 4500 50  0001 C CNN "LCSC"
-F 5 "GRM188R60J106KE47D" H 950 4500 50  0001 C CNN "Part Number"
+F 4 "C38898" H 950 4500 50  0001 C CNN "LCSC"
+F 5 "0603X106K100NT" H 950 4500 50  0001 C CNN "Part Number"
 	1    950  4500
 	1    0    0    -1
 $EndComp
+Text Label 5700 2900 2    50   ~ 0
+PA8
 Text Label 5700 2800 2    50   ~ 0
-PA8
+PA9
 Text Label 5700 2700 2    50   ~ 0
-PA9
-Text Label 5700 2600 2    50   ~ 0
 PA10
-Text Label 5700 2900 2    50   ~ 0
+Text Label 5700 3000 2    50   ~ 0
 PB15
-Text Label 5700 3000 2    50   ~ 0
+Text Label 5700 3100 2    50   ~ 0
 PB14
-Text Label 5700 3100 2    50   ~ 0
+Text Label 5700 3200 2    50   ~ 0
 PB13
+Text Label 5700 3500 2    50   ~ 0
+PB10
 Text Label 5700 3400 2    50   ~ 0
-PB10
+PB11
+Text Label 5700 3800 2    50   ~ 0
+PB0
+Text Label 5700 3600 2    50   ~ 0
+PB2
+Text Label 5700 3700 2    50   ~ 0
+PB1
+Text Label 5700 4300 2    50   ~ 0
+PA3
+Text Label 5700 4200 2    50   ~ 0
+PA4
+Text Label 5700 4100 2    50   ~ 0
+PA5
+Text Label 5700 4000 2    50   ~ 0
+PA6
+Text Label 5700 3900 2    50   ~ 0
+PA7
+Text Label 4350 4200 0    50   ~ 0
+PA1
+Text Label 4350 4100 0    50   ~ 0
+PA0
+Text Label 4350 3800 0    50   ~ 0
+PC13
+Text Label 4350 3900 0    50   ~ 0
+PC14
+Text Label 4350 3400 0    50   ~ 0
+PB6
+Text Label 4350 3500 0    50   ~ 0
+PB7
+Text Label 4350 3600 0    50   ~ 0
+PB8
+Text Label 4350 3700 0    50   ~ 0
+PB9
+Text Label 4350 3300 0    50   ~ 0
+PB5
+Text Label 4350 3200 0    50   ~ 0
+PB4
+Text Label 4350 3100 0    50   ~ 0
+PB3
+Text Label 4350 2800 0    50   ~ 0
+PA13
+Text Label 4350 2900 0    50   ~ 0
+PA14
+Text Label 4350 3000 0    50   ~ 0
+PA15
+Text Label 4350 4000 0    50   ~ 0
+PC15
 Text Label 5700 3300 2    50   ~ 0
-PB11
-Text Label 5700 3700 2    50   ~ 0
-PB0
-Text Label 5700 3500 2    50   ~ 0
-PB2
-Text Label 5700 3600 2    50   ~ 0
-PB1
-Text Label 5700 4200 2    50   ~ 0
-PA3
-Text Label 5700 4100 2    50   ~ 0
-PA4
-Text Label 5700 4000 2    50   ~ 0
-PA5
-Text Label 5700 3900 2    50   ~ 0
-PA6
-Text Label 5700 3800 2    50   ~ 0
-PA7
+PB12
 Text Label 4350 4300 0    50   ~ 0
-PA1
-Text Label 4350 4200 0    50   ~ 0
-PA0
-Text Label 4350 3900 0    50   ~ 0
-PC13
-Text Label 4350 4000 0    50   ~ 0
-PC14
-Text Label 4350 3500 0    50   ~ 0
-PB6
-Text Label 4350 3600 0    50   ~ 0
-PB7
-Text Label 4350 3700 0    50   ~ 0
-PB8
-Text Label 4350 3800 0    50   ~ 0
-PB9
-Text Label 4350 3400 0    50   ~ 0
-PB5
-Text Label 4350 3300 0    50   ~ 0
-PB4
-Text Label 4350 3200 0    50   ~ 0
-PB3
-Text Label 4350 2900 0    50   ~ 0
-PA13
-Text Label 4350 3000 0    50   ~ 0
-PA14
-Text Label 4350 3100 0    50   ~ 0
-PA15
-Text Label 4350 4100 0    50   ~ 0
-PC15
-Text Label 5700 3200 2    50   ~ 0
-PB12
-Text Label 5700 4300 2    50   ~ 0
 PA2
+Connection ~ 1200 1400
+Wire Wire Line
+	1200 1400 1200 1750
+Wire Notes Line
+	600  6400 4250 6400
+Wire Notes Line
+	600  7650 4250 7650
+$Comp
+L MCU_ST_STM32F1:STM32F103C8Tx U?
+U 1 1 5E5783D5
+P 7000 3100
+F 0 "U?" H 6950 1511 50  0000 C CNN
+F 1 "STM32F103C8Tx" H 6950 1420 50  0000 C CNN
+F 2 "Package_QFP:LQFP-48_7x7mm_P0.5mm" H 6400 1700 50  0001 R CNN
+F 3 "http://www.st.com/st-web-ui/static/active/en/resource/technical/document/datasheet/CD00161566.pdf" H 7000 3100 50  0001 C CNN
+	1    7000 3100
+	1    0    0    -1
+$EndComp
+Wire Notes Line
+	4250 6400 4250 7650
+Text Notes 2200 7550 0    50   ~ 0
+U don't need most of them if u use F103\n
 $EndSCHEMATC

Commit message: Appearently buy parts is hard
Parts:
- removed U?: STM32F103C8Tx, Package_QFP:LQFP-48_7x7mm_P0.5mm, symbol MCU_ST_STM32F1:STM32F103C8Tx
- C1, C5, C6, C7, C9: LCSC C307348 -> C80516; Part Number CL10B104KB8WPNC -> 0603B104K160CT
- R1: LCSC C116674 -> C100703; Part Number AC0603FR-07100KL -> CR0603FA1003G
- R2, R3: LCSC C114668 -> C103303; Part Number RC0603FR-071K5L -> RTT031501FTP
- Y1: value 8Mhz 20pf -> 8Mhz 10pf
Changed lines of the file:
@@
 F 2 "Capacitor_SMD:C_0603_1608Metric" H 2188 6850 50  0001 C CNN
 F 3 "~" H 2150 7000 50  0001 C CNN
-F 4 "C307348" H 2150 7000 50  0001 C CNN "LCSC"
-F 5 "CL10B104KB8WPNC" H 2150 7000 50  0001 C CNN "Part Number"
+F 4 "C80516" H 2150 7000 50  0001 C CNN "LCSC"
+F 5 "0603B104K160CT" H 2150 7000 50  0001 C CNN "Part Number"
 	1    2150 7000
 	1    0    0    -1
@@
 F 2 "Capacitor_SMD:C_0603_1608Metric" H 1738 6850 50  0001 C CNN
 F 3 "~" H 1700 7000 50  0001 C CNN
-F 4 "C307348" H 1700 7000 50  0001 C CNN "LCSC"
-F 5 "CL10B104KB8WPNC" H 1700 7000 50  0001 C CNN "Part Number"
+F 4 "C80516" H 1700 7000 50  0001 C CNN "LCSC"
+F 5 "0603B104K160CT" H 1700 7000 50  0001 C CNN "Part Number"
 	1    1700 7000
 	1    0    0    -1
@@
 F 2 "Capacitor_SMD:C_0603_1608Metric" H 1288 6850 50  0001 C CNN
 F 3 "~" H 1250 7000 50  0001 C CNN
-F 4 "C307348" H 1250 7000 50  0001 C CNN "LCSC"
-F 5 "CL10B104KB8WPNC" H 1250 7000 50  0001 C CNN "Part Number"
+F 4 "C80516" H 1250 7000 50  0001 C CNN "LCSC"
+F 5 "0603B104K160CT" H 1250 7000 50  0001 C CNN "Part Number"
 	1    1250 7000
 	1    0    0    -1
@@
 F 2 "Capacitor_SMD:C_0603_1608Metric" H 838 6850 50  0001 C CNN
 F 3 "~" H 800 7000 50  0001 C CNN
-F 4 "C307348" H 800 7000 50  0001 C CNN "LCSC"
-F 5 "CL10B104KB8WPNC" H 800 7000 50  0001 C CNN "Part Number"
+F 4 "C80516" H 800 7000 50  0001 C CNN "LCSC"
+F 5 "0603B104K160CT" H 800 7000 50  0001 C CNN "Part Number"
 	1    800  7000
 	1    0    0    -1
@@
 F 2 "Capacitor_SMD:C_0603_1608Metric" H 1238 1100 50  0001 C CNN
 F 3 "~" H 1200 1250 50  0001 C CNN
-F 4 "C307348" H 1200 1250 50  0001 C CNN "LCSC"
-F 5 "CL10B104KB8WPNC" H 1200 1250 50  0001 C CNN "Part Number"
+F 4 "C80516" H 1200 1250 50  0001 C CNN "LCSC"
+F 5 "0603B104K160CT" H 1200 1250 50  0001 C CNN "Part Number"
 	1    1200 1250
 	1    0    0    -1
@@
 F 2 "Resistor_SMD:R_0603_1608Metric" V 1530 3350 50  0001 C CNN
 F 3 "~" H 1600 3350 50  0001 C CNN
-F 4 "C114668" H 1600 3350 50  0001 C CNN "LCSC"
-F 5 "RC0603FR-071K5L" H 1600 3350 50  0001 C CNN "Part Number"
+F 4 "C103303" H 1600 3350 50  0001 C CNN "LCSC"
+F 5 "RTT031501FTP" H 1600 3350 50  0001 C CNN "Part Number"
 	1    1600 3350
 	1    0    0    -1
@@
 F 2 "Resistor_SMD:R_0603_1608Metric" V 730 1600 50  0001 C CNN
 F 3 "~" H 800 1600 50  0001 C CNN
-F 4 "C116674" H 800 1600 50  0001 C CNN "LCSC"
-F 5 "AC0603FR-07100KL" H 800 1600 50  0001 C CNN "Part Number"
+F 4 "C100703" H 800 1600 50  0001 C CNN "LCSC"
+F 5 "CR0603FA1003G" H 800 1600 50  0001 C CNN "Part Number"
 	1    800  1600
 	1    0    0    -1
@@
 F 2 "Resistor_SMD:R_0603_1608Metric" V 1580 5800 50  0001 C CNN
 F 3 "~" H 1650 5800 50  0001 C CNN
-F 4 "C114668" H 1650 5800 50  0001 C CNN "LCSC"
-F 5 "RC0603FR-071K5L" H 1650 5800 50  0001 C CNN "Part Number"
+F 4 "C103303" H 1650 5800 50  0001 C CNN "LCSC"
+F 5 "RTT031501FTP" H 1650 5800 50  0001 C CNN "Part Number"
 	1    1650 5800
 	0    1    1    0
@@
 P 1400 5650
 F 0 "Y1" V 1354 5894 50  0000 L CNN
-F 1 "8Mhz 20pf" V 1445 5894 50  0000 L CNN
+F 1 "8Mhz 10pf" V 1445 5894 50  0000 L CNN
 F 2 "Crystal:Crystal_SMD_3225-4Pin_3.2x2.5mm" H 1400 5650 50  0001 C CNN
 F 3 "https://datasheet.lcsc.com/szlcsc/1906261509_Zhejiang-Abel-Elec-TAXM8M4RDBCCT2T_C400090.pdf" H 1400 5650 50  0001 C CNN
@@
 Wire Notes Line
 	600  7650 4250 7650
-$Comp
-L MCU_ST_STM32F1:STM32F103C8Tx U?
-U 1 1 5E5783D5
-P 7000 3100
-F 0 "U?" H 6950 1511 50  0000 C CNN
-F 1 "STM32F103C8Tx" H 6950 1420 50  0000 C CNN
-F 2 "Package_QFP:LQFP-48_7x7mm_P0.5mm" H 6400 1700 50  0001 R CNN
-F 3 "http://www.st.com/st-web-ui/static/active/en/resource/technical/document/datasheet/CD00161566.pdf" H 7000 3100 50  0001 C CNN
-	1    7000 3100
-	1    0    0    -1
-$EndComp
 Wire Notes Line
 	4250 6400 4250 7650
